Commit message: добавлено 4 колесо

File: src/forklift_demo_description/urdf/forklift_demo.urdf.xacro (robot description, xacro)
@@ -60,5 +60,5 @@
     <parent link="base_link"/>
     <child link="rear_steer_link"/>
-    <origin xyz="-0.42 0.0 0.18" rpy="0 0 0"/>
+    <origin xyz="-0.42 0.35 0.18" rpy="0 0 0"/>
     <axis xyz="0 0 1"/>
     <limit effort="50" velocity="1.5" lower="-$(arg max_steering_angle)" upper="$(arg max_steering_angle)"/>
@@ -79,4 +79,26 @@
     <axis xyz="0 1 0"/>
   </joint>
+  <link name="rear_right_caster_link"/>
+  <joint name="rear_right_steering_joint" type="continuous">
+    <parent link="base_link"/>
+    <child link="rear_right_caster_link"/>
+    <origin xyz="-0.34 -0.35 0.18" rpy="0 0 0"/>
+    <axis xyz="0 0 1"/>
+  </joint>
+  <link name="rear_right_wheel_link">
+    <visual>
+      <origin xyz="0 0 0" rpy="1.57079632679 0 0"/>
+      <geometry>
+        <cylinder radius="$(arg wheel_radius)" length="0.10"/>
+      </geometry>
+      <material name="wheel_black"/>
+    </visual>
+  </link>
+  <joint name="rear_right_wheel_joint" type="continuous">
+    <parent link="rear_right_caster_link"/>
+    <child link="rear_right_wheel_link"/>
+    <origin xyz="-0.08 0 0" rpy="0 0 0"/>
+    <axis xyz="0 1 0"/>
+  </joint>
   <link name="laser_link">
     <visual>

Commit message: работает демо 4 колеса

File: src/forklift_demo_description/urdf/forklift_demo.urdf.xacro (robot description, xacro)
@@ -17,4 +17,7 @@
     <color rgba="0.12 0.12 0.12 1.0"/>
   </material>
+  <material name="fork_steel">
+    <color rgba="0.72 0.72 0.72 1.0"/>
+  </material>
   <link name="base_link">
     <visual>
@@ -24,4 +27,25 @@
       </geometry>
       <material name="body_orange"/>
+    </visual>
+    <visual>
+      <origin xyz="0.60 0 0.18" rpy="0 0 0"/>
+      <geometry>
+        <box size="0.08 0.46 0.18"/>
+      </geometry>
+      <material name="fork_steel"/>
+    </visual>
+    <visual>
+      <origin xyz="0.88 0.18 0.10" rpy="0 0 0"/>
+      <geometry>
+        <box size="0.56 0.08 0.04"/>
+      </geometry>
+      <material name="fork_steel"/>
+    </visual>
+    <visual>
+      <origin xyz="0.88 -0.18 0.10" rpy="0 0 0"/>
+      <geometry>
+        <box size="0.56 0.08 0.04"/>
+      </geometry>
+      <material name="fork_steel"/>
     </visual>
   </link>

Commit message: добвил скругления пути, обновил модель

File: src/forklift_demo_description/urdf/forklift_demo.urdf.xacro (robot description, xacro)
@@ -2,12 +2,15 @@
 <robot xmlns:xacro="http://www.ros.org/wiki/xacro" name="forklift_demo">
   <xacro:arg name="use_sim_time" default="true"/>
-  <xacro:arg name="base_length" default="1.2"/>
+  <xacro:arg name="base_length" default="0.36"/>
   <xacro:arg name="base_width" default="0.8"/>
   <xacro:arg name="base_height" default="0.32"/>
+  <xacro:arg name="body_x_offset" default="-0.38"/>
   <xacro:arg name="wheel_radius" default="0.18"/>
   <xacro:arg name="wheel_width" default="0.08"/>
+  <xacro:arg name="passive_wheel_radius" default="0.045"/>
+  <xacro:arg name="passive_wheel_width" default="0.02"/>
   <xacro:arg name="wheelbase" default="1.2"/>
   <xacro:arg name="max_steering_angle" default="1.48353"/>
-  <xacro:arg name="laser_x" default="0.2"/>
+  <xacro:arg name="laser_x" default="-0.38"/>
   <xacro:arg name="laser_z" default="0.55"/>
   <material name="body_orange">
@@ -22,5 +25,5 @@
   <link name="base_link">
     <visual>
-      <origin xyz="0 0 0.25" rpy="0 0 0"/>
+      <origin xyz="$(arg body_x_offset) 0 0.25" rpy="0 0 0"/>
       <geometry>
         <box size="$(arg base_length) $(arg base_width) $(arg base_height)"/>
@@ -29,21 +32,14 @@
     </visual>
     <visual>
-      <origin xyz="0.60 0 0.18" rpy="0 0 0"/>
+      <origin xyz="0.36 0.35 0.10" rpy="0 0 0"/>
       <geometry>
-        <box size="0.08 0.46 0.18"/>
+        <box size="1.12 0.14 0.04"/>
       </geometry>
       <material name="fork_steel"/>
     </visual>
     <visual>
-      <origin xyz="0.88 0.18 0.10" rpy="0 0 0"/>
+      <origin xyz="0.36 -0.35 0.10" rpy="0 0 0"/>
       <geometry>
-        <box size="0.56 0.08 0.04"/>
-      </geometry>
-      <material name="fork_steel"/>
-    </visual>
-    <visual>
-      <origin xyz="0.88 -0.18 0.10" rpy="0 0 0"/>
-      <geometry>
-        <box size="0.56 0.08 0.04"/>
+        <box size="1.12 0.14 0.04"/>
       </geometry>
       <material name="fork_steel"/>
@@ -54,5 +50,5 @@
       <origin xyz="0 0 0" rpy="1.57079632679 0 0"/>
       <geometry>
-        <cylinder radius="$(arg wheel_radius)" length="$(arg wheel_width)"/>
+        <cylinder radius="$(arg passive_wheel_radius)" length="$(arg passive_wheel_width)"/>
       </geometry>
       <material name="wheel_black"/>
@@ -63,5 +59,5 @@
       <origin xyz="0 0 0" rpy="1.57079632679 0 0"/>
       <geometry>
-        <cylinder radius="$(arg wheel_radius)" length="$(arg wheel_width)"/>
+        <cylinder radius="$(arg passive_wheel_radius)" length="$(arg passive_wheel_width)"/>
       </geometry>
       <material name="wheel_black"/>
@@ -71,5 +67,5 @@
     <parent link="base_link"/>
     <child link="front_left_wheel_link"/>
-    <origin xyz="0.42 0.35 0.18" rpy="0 0 0"/>
+    <origin xyz="0.42 0.35 0.045" rpy="0 0 0"/>
     <axis xyz="0 1 0"/>
   </joint>
@@ -77,5 +73,5 @@
     <parent link="base_link"/>
     <child link="front_right_wheel_link"/>
-    <origin xyz="0.42 -0.35 0.18" rpy="0 0 0"/>
+    <origin xyz="0.42 -0.35 0.045" rpy="0 0 0"/>
     <axis xyz="0 1 0"/>
   </joint>

Commit message: перевозит палету с места на место

File: src/forklift_demo_description/urdf/forklift_demo.urdf.xacro (robot description, xacro)
@@ -8,8 +8,8 @@
   <xacro:arg name="wheel_radius" default="0.18"/>
   <xacro:arg name="wheel_width" default="0.08"/>
-  <xacro:arg name="passive_wheel_radius" default="0.045"/>
+  <xacro:arg name="passive_wheel_radius" default="0.03"/>
   <xacro:arg name="passive_wheel_width" default="0.02"/>
   <xacro:arg name="wheelbase" default="1.2"/>
-  <xacro:arg name="max_steering_angle" default="1.48353"/>
+  <xacro:arg name="max_steering_angle" default="1.57079632679"/>
   <xacro:arg name="laser_x" default="-0.38"/>
   <xacro:arg name="laser_z" default="0.55"/>
@@ -31,19 +31,28 @@
       <material name="body_orange"/>
     </visual>
+  </link>
+  <link name="fork_carriage_link">
     <visual>
-      <origin xyz="0.36 0.35 0.10" rpy="0 0 0"/>
+      <origin xyz="0.36 0.135 0.04" rpy="0 0 0"/>
       <geometry>
-        <box size="1.12 0.14 0.04"/>
+        <box size="1.12 0.06 0.04"/>
       </geometry>
       <material name="fork_steel"/>
     </visual>
     <visual>
-      <origin xyz="0.36 -0.35 0.10" rpy="0 0 0"/>
+      <origin xyz="0.36 -0.135 0.04" rpy="0 0 0"/>
       <geometry>
-        <box size="1.12 0.14 0.04"/>
+        <box size="1.12 0.06 0.04"/>
       </geometry>
       <material name="fork_steel"/>
     </visual>
   </link>
+  <joint name="fork_lift_joint" type="prismatic">
+    <parent link="base_link"/>
+    <child link="fork_carriage_link"/>
+    <origin xyz="0 0 0" rpy="0 0 0"/>
+    <axis xyz="0 0 1"/>
+    <limit effort="5000" velocity="0.4" lower="0.0" upper="0.28"/>
+  </joint>
   <link name="front_left_wheel_link">
     <visual>
@@ -67,5 +76,5 @@
     <parent link="base_link"/>
     <child link="front_left_wheel_link"/>
-    <origin xyz="0.42 0.35 0.045" rpy="0 0 0"/>
+    <origin xyz="0.42 0.135 0.03" rpy="0 0 0"/>
     <axis xyz="0 1 0"/>
   </joint>
@@ -73,5 +82,5 @@
     <parent link="base_link"/>
     <child link="front_right_wheel_link"/>
-    <origin xyz="0.42 -0.35 0.045" rpy="0 0 0"/>
+    <origin xyz="0.42 -0.135 0.03" rpy="0 0 0"/>
     <axis xyz="0 1 0"/>
   </joint>

Commit message: Добавлено новое управление для низкоуровневого контроллера, заменив старый `cmd_vel_to_tricycle` на `cmd_vel_to_motors`. Обновлены конфигурации и добавлены новые зависимости для `rqt_robot_steering`. Обновлены параметры навигации и модели, включая новые камеры и изменения в SDF.

File: src/forklift_demo_description/urdf/forklift_demo.urdf.xacro (robot description, xacro)
@@ -10,8 +10,10 @@
   <xacro:arg name="passive_wheel_radius" default="0.03"/>
   <xacro:arg name="passive_wheel_width" default="0.02"/>
-  <xacro:arg name="wheelbase" default="1.2"/>
+  <xacro:arg name="wheelbase" default="0.84"/>
   <xacro:arg name="max_steering_angle" default="1.57079632679"/>
   <xacro:arg name="laser_x" default="-0.38"/>
   <xacro:arg name="laser_z" default="0.55"/>
+  <xacro:arg name="fork_depth_camera_x" default="-0.24"/>
+  <xacro:arg name="fork_depth_camera_z" default="0.14"/>
   <material name="body_orange">
     <color rgba="0.90 0.62 0.18 1.0"/>
@@ -32,4 +34,10 @@
     </visual>
   </link>
+  <link name="tracking_link"/>
+  <joint name="tracking_joint" type="fixed">
+    <parent link="base_link"/>
+    <child link="tracking_link"/>
+    <origin xyz="0.42 0 0" rpy="0 0 0"/>
+  </joint>
   <link name="fork_carriage_link">
     <visual>
@@ -91,5 +99,5 @@
     <origin xyz="-0.42 0.35 0.18" rpy="0 0 0"/>
     <axis xyz="0 0 1"/>
-    <limit effort="50" velocity="1.5" lower="-$(arg max_steering_angle)" upper="$(arg max_steering_angle)"/>
+    <limit effort="120" velocity="2.0" lower="-$(arg max_steering_angle)" upper="$(arg max_steering_angle)"/>
   </joint>
   <link name="rear_drive_wheel_link">
@@ -107,4 +115,5 @@
     <origin xyz="0 0 0" rpy="0 0 0"/>
     <axis xyz="0 1 0"/>
+    <limit effort="800" velocity="12.0"/>
   </joint>
   <link name="rear_right_caster_link"/>
@@ -144,3 +153,17 @@
     <origin xyz="$(arg laser_x) 0 $(arg laser_z)" rpy="0 0 0"/>
   </joint>
+  <link name="fork_depth_camera_link">
+    <visual>
+      <origin xyz="0 0 0" rpy="0 0 0"/>
+      <geometry>
+        <box size="0.08 0.04 0.04"/>
+      </geometry>
+      <material name="wheel_black"/>
+    </visual>
+  </link>
+  <joint name="fork_depth_camera_joint" type="fixed">
+    <parent link="base_link"/>
+    <child link="fork_depth_camera_link"/>
+    <origin xyz="$(arg fork_depth_camera_x) 0 $(arg fork_depth_camera_z)" rpy="0 0 0"/>
+  </joint>
 </robot>

Commit message: Refactor Docker setup and remove unused components. Updated docker-compose.yml to streamline service configurations and added volume mappings. Enhanced Dockerfile for improved package installation with retry logic. Removed deprecated nodes and services from the forklift demo control package, focusing on the route-server navigation stack. Updated README for clarity on system architecture and removed references to deleted components.

File: src/forklift_demo_description/urdf/forklift_demo.urdf.xacro (robot description, xacro)
@@ -14,6 +14,4 @@
   <xacro:arg name="laser_x" default="-0.38"/>
   <xacro:arg name="laser_z" default="0.55"/>
-  <xacro:arg name="fork_depth_camera_x" default="-0.24"/>
-  <xacro:arg name="fork_depth_camera_z" default="0.14"/>
   <material name="body_orange">
     <color rgba="0.90 0.62 0.18 1.0"/>
@@ -153,17 +151,3 @@
     <origin xyz="$(arg laser_x) 0 $(arg laser_z)" rpy="0 0 0"/>
   </joint>
-  <link name="fork_depth_camera_link">
-    <visual>
-      <origin xyz="0 0 0" rpy="0 0 0"/>
-      <geometry>
-        <box size="0.08 0.04 0.04"/>
-      </geometry>
-      <material name="wheel_black"/>
-    </visual>
-  </link>
-  <joint name="fork_depth_camera_joint" type="fixed">
-    <parent link="base_link"/>
-    <child link="fork_depth_camera_link"/>
-    <origin xyz="$(arg fork_depth_camera_x) 0 $(arg fork_depth_camera_z)" rpy="0 0 0"/>
-  </joint>
 </robot>

Commit message: Add RQT container for robot steering and update dependencies. Enhanced Docker setup with new service in docker-compose.yml for `rqt_robot_steering`. Updated Dockerfile to include necessary ROS packages. Adjusted various configuration files to replace `tracking_link` with `base_link` for consistency across the project. Improved README to reflect new RQT usage instructions.

File: src/forklift_demo_description/urdf/forklift_demo.urdf.xacro (robot description, xacro)
@@ -23,7 +23,8 @@
     <color rgba="0.72 0.72 0.72 1.0"/>
   </material>
-  <link name="base_link">
+  <link name="base_link"/>
+  <link name="chassis_link">
     <visual>
-      <origin xyz="$(arg body_x_offset) 0 0.25" rpy="0 0 0"/>
+      <origin xyz="0.80 0 0.25" rpy="0 0 0"/>
       <geometry>
         <box size="$(arg base_length) $(arg base_width) $(arg base_height)"/>
@@ -32,9 +33,8 @@
     </visual>
   </link>
-  <link name="tracking_link"/>
-  <joint name="tracking_joint" type="fixed">
+  <joint name="base_to_chassis_joint" type="fixed">
     <parent link="base_link"/>
-    <child link="tracking_link"/>
-    <origin xyz="0.42 0 0" rpy="0 0 0"/>
+    <child link="chassis_link"/>
+    <origin xyz="0 0 0" rpy="0 0 0"/>
   </joint>
   <link name="fork_carriage_link">
@@ -55,7 +55,7 @@
   </link>
   <joint name="fork_lift_joint" type="prismatic">
-    <parent link="base_link"/>
+    <parent link="chassis_link"/>
     <child link="fork_carriage_link"/>
-    <origin xyz="0 0 0" rpy="0 0 0"/>
+    <origin xyz="0.42 0 0" rpy="0 0 3.14159265359"/>
     <axis xyz="0 0 1"/>
     <limit effort="5000" velocity="0.4" lower="0.0" upper="0.28"/>
@@ -80,20 +80,20 @@
   </link>
   <joint name="front_left_wheel_joint" type="continuous">
-    <parent link="base_link"/>
+    <parent link="chassis_link"/>
     <child link="front_left_wheel_link"/>
-    <origin xyz="0.42 0.135 0.03" rpy="0 0 0"/>
-    <axis xyz="0 1 0"/>
+    <origin xyz="0 -0.135 0.03" rpy="0 0 3.14159265359"/>
+    <axis xyz="0 -1 0"/>
   </joint>
   <joint name="front_right_wheel_joint" type="continuous">
-    <parent link="base_link"/>
+    <parent link="chassis_link"/>
     <child link="front_right_wheel_link"/>
-    <origin xyz="0.42 -0.135 0.03" rpy="0 0 0"/>
-    <axis xyz="0 1 0"/>
+    <origin xyz="0 0.135 0.03" rpy="0 0 3.14159265359"/>
+    <axis xyz="0 -1 0"/>
   </joint>
   <link name="rear_steer_link"/>
   <joint name="rear_steering_joint" type="revolute">
-    <parent link="base_link"/>
+    <parent link="chassis_link"/>
     <child link="rear_steer_link"/>
-    <origin xyz="-0.42 0.35 0.18" rpy="0 0 0"/>
+    <origin xyz="0.84 -0.35 0.18" rpy="0 0 3.14159265359"/>
     <axis xyz="0 0 1"/>
     <limit effort="120" velocity="2.0" lower="-$(arg max_steering_angle)" upper="$(arg max_steering_angle)"/>
@@ -112,12 +112,12 @@
     <child link="rear_drive_wheel_link"/>
     <origin xyz="0 0 0" rpy="0 0 0"/>
-    <axis xyz="0 1 0"/>
+    <axis xyz="0 -1 0"/>
     <limit effort="800" velocity="12.0"/>
   </joint>
   <link name="rear_right_caster_link"/>
   <joint name="rear_right_steering_joint" type="continuous">
-    <parent link="base_link"/>
+    <parent link="chassis_link"/>
     <child link="rear_right_caster_link"/>
-    <origin xyz="-0.34 -0.35 0.18" rpy="0 0 0"/>
+    <origin xyz="0.76 0.35 0.18" rpy="0 0 3.14159265359"/>
     <axis xyz="0 0 1"/>
   </joint>
@@ -135,5 +135,5 @@
     <child link="rear_right_wheel_link"/>
     <origin xyz="-0.08 0 0" rpy="0 0 0"/>
-    <axis xyz="0 1 0"/>
+    <axis xyz="0 -1 0"/>
   </joint>
   <link name="laser_link">
@@ -147,7 +147,7 @@
   </link>
   <joint name="laser_joint" type="fixed">
-    <parent link="base_link"/>
+    <parent link="chassis_link"/>
     <child link="laser_link"/>
-    <origin xyz="$(arg laser_x) 0 $(arg laser_z)" rpy="0 0 0"/>
+    <origin xyz="0.80 0 $(arg laser_z)" rpy="0 0 0"/>
   </joint>
 </robot>
