Commit message: Remove forklift_urdf package and associated files, including CMakeLists.txt, package.xml, configuration, launch files, URDF, and mesh assets. Update forklift_demo_control to include a new fork position controller and adjust cmd_vel_to_motors parameters for right steering and wheel commands. Enhance bridge configuration with additional Lidar topics and update navigation parameters for improved collision monitoring and mapping. Modify RViz configuration for better visualization of Lidar data.

File: src/forklift_demo_description/urdf/forklift_demo.urdf.xacro (robot description, xacro)
@@ -1,153 +1,961 @@
-<?xml version="1.0"?>
+<?xml version="1.0" encoding="utf-8"?>
+<!-- This URDF was automatically created by SolidWorks to URDF Exporter! Originally created by Stephen Brawner (brawner@gmail.com)
+     Commit Version: 1.6.0-4-g7f85cfe  Build Version: 1.6.7995.38578
+     For more information, please see http://wiki.ros.org/sw_urdf_exporter -->
 <robot xmlns:xacro="http://www.ros.org/wiki/xacro" name="forklift_demo">
   <xacro:arg name="use_sim_time" default="true"/>
-  <xacro:arg name="base_length" default="0.36"/>
-  <xacro:arg name="base_width" default="0.8"/>
-  <xacro:arg name="base_height" default="0.32"/>
-  <xacro:arg name="body_x_offset" default="-0.38"/>
-  <xacro:arg name="wheel_radius" default="0.18"/>
-  <xacro:arg name="wheel_width" default="0.08"/>
-  <xacro:arg name="passive_wheel_radius" default="0.03"/>
-  <xacro:arg name="passive_wheel_width" default="0.02"/>
-  <xacro:arg name="wheelbase" default="0.84"/>
-  <xacro:arg name="max_steering_angle" default="1.57079632679"/>
-  <xacro:arg name="laser_x" default="-0.38"/>
-  <xacro:arg name="laser_z" default="0.55"/>
-  <material name="body_orange">
-    <color rgba="0.90 0.62 0.18 1.0"/>
-  </material>
-  <material name="wheel_black">
-    <color rgba="0.12 0.12 0.12 1.0"/>
-  </material>
-  <material name="fork_steel">
-    <color rgba="0.72 0.72 0.72 1.0"/>
-  </material>
-  <link name="base_link"/>
-  <link name="chassis_link">
-    <visual>
-      <origin xyz="0.80 0 0.25" rpy="0 0 0"/>
-      <geometry>
-        <box size="$(arg base_length) $(arg base_width) $(arg base_height)"/>
-      </geometry>
-      <material name="body_orange"/>
-    </visual>
-  </link>
-  <joint name="base_to_chassis_joint" type="fixed">
-    <parent link="base_link"/>
-    <child link="chassis_link"/>
-    <origin xyz="0 0 0" rpy="0 0 0"/>
-  </joint>
-  <link name="fork_carriage_link">
-    <visual>
-      <origin xyz="0.36 0.135 0.04" rpy="0 0 0"/>
-      <geometry>
-        <box size="1.12 0.06 0.04"/>
-      </geometry>
-      <material name="fork_steel"/>
-    </visual>
-    <visual>
-      <origin xyz="0.36 -0.135 0.04" rpy="0 0 0"/>
-      <geometry>
-        <box size="1.12 0.06 0.04"/>
-      </geometry>
-      <material name="fork_steel"/>
-    </visual>
-  </link>
-  <joint name="fork_lift_joint" type="prismatic">
-    <parent link="chassis_link"/>
-    <child link="fork_carriage_link"/>
-    <origin xyz="0.42 0 0" rpy="0 0 3.14159265359"/>
-    <axis xyz="0 0 1"/>
-    <limit effort="5000" velocity="0.4" lower="0.0" upper="0.28"/>
-  </joint>
-  <link name="front_left_wheel_link">
-    <visual>
-      <origin xyz="0 0 0" rpy="1.57079632679 0 0"/>
-      <geometry>
-        <cylinder radius="$(arg passive_wheel_radius)" length="$(arg passive_wheel_width)"/>
-      </geometry>
-      <material name="wheel_black"/>
-    </visual>
-  </link>
-  <link name="front_right_wheel_link">
-    <visual>
-      <origin xyz="0 0 0" rpy="1.57079632679 0 0"/>
-      <geometry>
-        <cylinder radius="$(arg passive_wheel_radius)" length="$(arg passive_wheel_width)"/>
-      </geometry>
-      <material name="wheel_black"/>
-    </visual>
-  </link>
-  <joint name="front_left_wheel_joint" type="continuous">
-    <parent link="chassis_link"/>
-    <child link="front_left_wheel_link"/>
-    <origin xyz="0 -0.135 0.03" rpy="0 0 3.14159265359"/>
-    <axis xyz="0 -1 0"/>
-  </joint>
-  <joint name="front_right_wheel_joint" type="continuous">
-    <parent link="chassis_link"/>
-    <child link="front_right_wheel_link"/>
-    <origin xyz="0 0.135 0.03" rpy="0 0 3.14159265359"/>
-    <axis xyz="0 -1 0"/>
-  </joint>
-  <link name="rear_steer_link"/>
-  <joint name="rear_steering_joint" type="revolute">
-    <parent link="chassis_link"/>
-    <child link="rear_steer_link"/>
-    <origin xyz="0.84 -0.35 0.18" rpy="0 0 3.14159265359"/>
-    <axis xyz="0 0 1"/>
-    <limit effort="120" velocity="2.0" lower="-$(arg max_steering_angle)" upper="$(arg max_steering_angle)"/>
-  </joint>
-  <link name="rear_drive_wheel_link">
-    <visual>
-      <origin xyz="0 0 0" rpy="1.57079632679 0 0"/>
-      <geometry>
-        <cylinder radius="$(arg wheel_radius)" length="0.10"/>
-      </geometry>
-      <material name="wheel_black"/>
-    </visual>
-  </link>
-  <joint name="rear_wheel_joint" type="continuous">
-    <parent link="rear_steer_link"/>
-    <child link="rear_drive_wheel_link"/>
-    <origin xyz="0 0 0" rpy="0 0 0"/>
-    <axis xyz="0 -1 0"/>
-    <limit effort="800" velocity="12.0"/>
-  </joint>
-  <link name="rear_right_caster_link"/>
-  <joint name="rear_right_steering_joint" type="continuous">
-    <parent link="chassis_link"/>
-    <child link="rear_right_caster_link"/>
-    <origin xyz="0.76 0.35 0.18" rpy="0 0 3.14159265359"/>
-    <axis xyz="0 0 1"/>
-  </joint>
-  <link name="rear_right_wheel_link">
-    <visual>
-      <origin xyz="0 0 0" rpy="1.57079632679 0 0"/>
-      <geometry>
-        <cylinder radius="$(arg wheel_radius)" length="0.10"/>
-      </geometry>
-      <material name="wheel_black"/>
-    </visual>
-  </link>
-  <joint name="rear_right_wheel_joint" type="continuous">
-    <parent link="rear_right_caster_link"/>
-    <child link="rear_right_wheel_link"/>
-    <origin xyz="-0.08 0 0" rpy="0 0 0"/>
-    <axis xyz="0 -1 0"/>
-  </joint>
-  <link name="laser_link">
-    <visual>
-      <origin xyz="0 0 0" rpy="0 0 0"/>
-      <geometry>
-        <cylinder radius="0.05" length="0.04"/>
-      </geometry>
-      <material name="wheel_black"/>
-    </visual>
-  </link>
-  <joint name="laser_joint" type="fixed">
-    <parent link="chassis_link"/>
-    <child link="laser_link"/>
-    <origin xyz="0.80 0 $(arg laser_z)" rpy="0 0 0"/>
-  </joint>
+  <link
+    name="base_link">
+    <inertial>
+      <origin
+        xyz="0.94148 -7.6988E-08 0.92711"
+        rpy="0 0 0" />
+      <mass
+        value="1000" />
+      <inertia
+        ixx="1152.4"
+        ixy="0.00030978"
+        ixz="23.035"
+        iyy="1102.3"
+        iyz="-5.1614E-05"
+        izz="320.85" />
+    </inertial>
+    <visual>
+      <origin
+        xyz="0 0 0"
+        rpy="0 0 0" />
+      <geometry>
+        <mesh
+          filename="package://forklift_demo_description/urdf/meshes/base_link.STL" />
+      </geometry>
+      <material
+        name="">
+        <color
+          rgba="0.10 0.75 1.00 1" />
+      </material>
+    </visual>
+  </link>
+  <link
+    name="left_lidar_link">
+    <inertial>
+      <origin
+        xyz="-6.9389E-18 0 6.9389E-18"
+        rpy="0 0 0" />
+      <mass
+        value="0.28464" />
+      <inertia
+        ixx="4.8105E-05"
+        ixy="-4.5139E-36"
+        ixz="9.5557E-09"
+        iyy="4.8105E-05"
+        iyz="9.2387E-38"
+        izz="6.8884E-05" />
+    </inertial>
+    <visual>
+      <origin
+        xyz="0 0 0"
+        rpy="0 0 0" />
+      <geometry>
+        <mesh
+          filename="package://forklift_demo_description/urdf/meshes/left_lidar_link.STL" />
+      </geometry>
+      <material
+        name="">
+        <color
+          rgba="0.10 0.75 1.00 1" />
+      </material>
+    </visual>
+    <collision>
+      <origin
+        xyz="0 0 0"
+        rpy="0 0 0" />
+      <geometry>
+        <mesh
+          filename="package://forklift_demo_description/urdf/meshes/left_lidar_link.STL" />
+      </geometry>
+    </collision>
+  </link>
+  <joint
+    name="left_lidar_joint"
+    type="fixed">
+    <origin
+      xyz="1.27295476942974 0.418116775610435 0.0239999999999846"
+      rpy="0 -0.000459874311882969 0" />
+    <parent
+      link="base_link" />
+    <child
+      link="left_lidar_link" />
+  </joint>
+  <link
+    name="right_lidar_link">
+    <inertial>
+      <origin
+        xyz="-6.9389E-18 -5.5511E-17 6.9389E-18"
+        rpy="0 0 0" />
+      <mass
+        value="0.28464" />
+      <inertia
+        ixx="4.8105E-05"
+        ixy="6.6884E-53"
+        ixz="3.7885E-22"
+        iyy="4.8105E-05"
+        iyz="1.4522E-37"
+        izz="6.8884E-05" />
+    </inertial>
+    <visual>
+      <origin
+        xyz="0 0 0"
+        rpy="0 0 0" />
+      <geometry>
+        <mesh
+          filename="package://forklift_demo_description/urdf/meshes/right_lidar_link.STL" />
+      </geometry>
+      <material
+        name="">
+        <color
+          rgba="1.00 0.18 0.70 1" />
+      </material>
+    </visual>
+    <collision>
+      <origin
+        xyz="0 0 0"
+        rpy="0 0 0" />
+      <geometry>
+        <mesh
+          filename="package://forklift_demo_description/urdf/meshes/right_lidar_link.STL" />
+      </geometry>
+    </collision>
+  </link>
+  <joint
+    name="right_lidar_joint"
+    type="fixed">
+    <origin
+      xyz="1.27295476942975 -0.418116775610423 0.0239999999999846"
+      rpy="0 0 0" />
+    <parent
+      link="base_link" />
+    <child
+      link="right_lidar_link" />
+  </joint>
+  <link
+    name="rear_lidar_link">
+    <inertial>
+      <origin
+        xyz="0 0 0.012"
+        rpy="0 0 0" />
+      <mass
+        value="0.28464" />
+      <inertia
+        ixx="4.8105E-05"
+        ixy="-6.0185E-36"
+        ixz="6.2789E-37"
+        iyy="4.8105E-05"
+        iyz="-2.0758E-37"
+        izz="6.8884E-05" />
+    </inertial>
+    <visual>
+      <origin
+        xyz="0 0 0"
+        rpy="0 0 0" />
+      <geometry>
+        <mesh
+          filename="package://forklift_demo_description/urdf/meshes/rear_lidar_link.STL" />
+      </geometry>
+      <material
+        name="">
+        <color
+          rgba="1.00 0.55 0.05 1" />
+      </material>
+    </visual>
+    <collision>
+      <origin
+        xyz="0 0 0"
+        rpy="0 0 0" />
+      <geometry>
+        <mesh
+          filename="package://forklift_demo_description/urdf/meshes/rear_lidar_link.STL" />
+      </geometry>
+    </collision>
+  </link>
+  <joint
+    name="rear_lidar_joint"
+    type="fixed">
+    <origin
+      xyz="0.705969649244955 0 0.0559999999999846"
+      rpy="0 0.000459874311882969 -3.14159265358978" />
+    <parent
+      link="base_link" />
+    <child
+      link="rear_lidar_link" />
+    <axis
+      xyz="0 0 0" />
+  </joint>
+  <link
+    name="up_lidar_link">
+    <inertial>
+      <origin
+        xyz="0 0 0"
+        rpy="0 0 0" />
+      <mass
+        value="0.284643374059973" />
+      <inertia
+        ixx="4.81274052613001E-05"
+        ixy="1.31890466162261E-35"
+        ixz="6.86039242171329E-07"
+        iyy="4.81047302161354E-05"
+        iyz="-3.03755087092172E-36"
+        izz="6.88610214773487E-05" />
+    </inertial>
+    <visual>
+      <origin
+        xyz="0 0 0"
+        rpy="0 0 0" />
+      <geometry>
+        <mesh
+          filename="package://forklift_demo_description/urdf/meshes/up_lidar_link.STL" />
+      </geometry>
+      <material
+        name="">
+        <color
+          rgba="0.792156862745098 0.819607843137255 0.933333333333333 1" />
+      </material>
+    </visual>
+    <collision>
+      <origin
+        xyz="0 0 0"
+        rpy="0 0 0" />
+      <geometry>
+        <mesh
+          filename="package://forklift_demo_description/urdf/meshes/up_lidar_link.STL" />
+      </geometry>
+    </collision>
+  </link>
+  <joint
+    name="up_lidar_joint"
+    type="fixed">
+    <origin
+      xyz="1.12608148221207 0 1.98742227080532"
+      rpy="0 -0.0334999573301522 0" />
+    <parent
+      link="base_link" />
+    <child
+      link="up_lidar_link" />
+    <axis
+      xyz="0 0 0" />
+  </joint>
+  <link
+    name="3d_lidar_link">
+    <inertial>
+      <origin
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
Commit message: Add fork_slider service to docker-compose for enhanced forklift demo functionality. Update Dockerfile to include ros-jazzy-slider-publisher dependency. Adjust route_server_params.yaml to modify smoothing_radius for improved path planning. Update sim_followpath.launch.py to include invert_position_command parameter. Refine euro_pallet model SDF for collision adjustments and update forklift_demo URDF to include collision geometry for fork_link.

File: src/forklift_demo_description/urdf/forklift_demo.urdf.xacro (robot description, xacro)
@@ -433,4 +433,13 @@
       </material>
     </visual>
+    <collision>
+      <origin
+        xyz="0 0 0"
+        rpy="0 0 0" />
+      <geometry>
+        <mesh
+          filename="package://forklift_demo_description/urdf/meshes/fork_link.STL" />
+      </geometry>
+    </collision>
   </link>
   <joint
@@ -445,5 +454,5 @@
       link="fork_link" />
     <axis
-      xyz="0 0 -1" />
+      xyz="0 0 1" />
     <limit
       lower="0"

Commit message: Refactor cmd_vel_activity_service and cmd_vel_to_motors to use wheel velocity commands instead of cmd_vel. Update parameters and subscriptions accordingly. Enhance steering alignment logic in cmd_vel_to_motors for improved control. Modify sim_followpath.launch.py to reflect changes in topic names.

File: src/forklift_demo_description/urdf/forklift_demo.urdf.xacro (robot description, xacro)
@@ -680,5 +680,5 @@
       lower="-3.1416"
       upper="3.1416"
-      effort="2500"
+      effort="1000000000"
       velocity="6.0" />
   </joint>
@@ -718,6 +718,5 @@
         rpy="0 0 0" />
       <geometry>
-        <mesh
-          filename="package://forklift_demo_description/urdf/meshes/right_wheel_link.STL" />
+        <cylinder radius="0.1" length="0.01" />
       </geometry>
     </collision>
@@ -955,6 +954,4 @@
       <i_max>5</i_max>
       <i_min>-5</i_min>
-      <cmd_max>120</cmd_max>
-      <cmd_min>-120</cmd_min>
     </plugin>
     <plugin filename="gz-sim-joint-controller-system" name="gz::sim::systems::JointController">

Commit message: Refactor RViz configuration and update URDF collision geometries for forklift demo. Removed unnecessary display panels in demo.rviz and replaced mesh collision geometries with cylinder shapes in forklift_demo.urdf.xacro for improved performance and simplicity.

File: src/forklift_demo_description/urdf/forklift_demo.urdf.xacro (robot description, xacro)
@@ -332,6 +332,5 @@
         rpy="0 0 0" />
       <geometry>
-        <mesh
-          filename="package://forklift_demo_description/urdf/meshes/fork_left_wheel_link.STL" />
+        <cylinder radius="0.04" length="0.07" />
       </geometry>
     </collision>
@@ -349,4 +348,7 @@
     <axis
       xyz="0 0 1" />
+    <dynamics
+      damping="0.0"
+      friction="0.0" />
   </joint>
   <link
@@ -385,6 +387,5 @@
         rpy="0 0 0" />
       <geometry>
-        <mesh
-          filename="package://forklift_demo_description/urdf/meshes/fork_right_wheel_link.STL" />
+        <cylinder radius="0.04" length="0.07" />
       </geometry>
     </collision>
@@ -402,4 +403,7 @@
     <axis
       xyz="0 0 1" />
+    <dynamics
+      damping="0.0"
+      friction="0.0" />
   </joint>
   <link
@@ -569,6 +573,9 @@
       lower="-3.1416"
       upper="3.1416"
-      effort="30"
+      effort="1000000000"
       velocity="6.0" />
+    <dynamics
+      damping="0.0"
+      friction="0.0" />
   </joint>
   <link
@@ -607,6 +614,5 @@
         rpy="0 0 0" />
       <geometry>
-        <mesh
-          filename="package://forklift_demo_description/urdf/meshes/left_wheel_link.STL" />
+        <cylinder radius="0.1" length="0.02" />
       </geometry>
     </collision>
@@ -624,4 +630,7 @@
     <axis
       xyz="0 0 1" />
+    <dynamics
+      damping="0.0"
+      friction="0.0" />
   </joint>
   <link
@@ -718,5 +727,5 @@
         rpy="0 0 0" />
       <geometry>
-        <cylinder radius="0.1" length="0.01" />
+        <cylinder radius="0.125" length="0.01" />
       </geometry>
     </collision>
